Commit message: Camera and Lidar are added

File: roverjw_description/urdf/RoverJW.xacro (robot description, xacro)
@@ -3,6 +3,7 @@
   <!-- Importing external urdf/xacros. -->
 	<xacro:include filename="$(find roverjw_description)/urdf/materials.xacro" />
-  	<xacro:include filename="$(find roverjw_description)/urdf/RoverJW.gazebo" />
+  <xacro:include filename="$(find roverjw_description)/urdf/RoverJW.gazebo" />
 	<xacro:include filename="$(find roverjw_description)/urdf/macros.xacro" />
+  <xacro:property name="cameraMass" value="0.1"/>
   <!-- Defining macros. -->
 	<xacro:macro name="wheel" params="prefix reflect_x:=1 reflect_y:=1 mimic:=false">
@@ -93,6 +94,5 @@
   <!-- Defining model links. -->
 	<link name="odom" />
-  <link
-    name="base_link">
+  <link name="base_link">
     <inertial>
       <origin
@@ -117,13 +117,12 @@
     <collision>
       <origin
-        xyz="0 0 0.15"
-        rpy="0 0 0" />
-      <geometry>
-        <box size="0.455 0.426 0.32" />
+        xyz="0 0 0.05"
+        rpy="0 0 0" />
+      <geometry>
+        <box size="0.455 0.426 0.16" />
       </geometry>
     </collision>
   </link>
-  <link
-    name="top_link">
+  <link name="top_link">
     <inertial>
       <origin
@@ -147,6 +146,5 @@
     </visual>
   </link>
-  <link
-    name="battery_link">
+  <link name="battery_link">
     <inertial>
       <origin
@@ -170,6 +168,5 @@
     </visual>
   </link>
-  <link
-    name="housing_link">
+  <link name="housing_link">
     <inertial>
       <origin
@@ -194,13 +191,9 @@
   </link>
   <!-- Defining model joints. -->
-  <joint
-    name="fixed_base_joint"
-    type="fixed">
+  <joint name="fixed_base_joint" type="fixed">
     <parent link="odom" />
     <child link="base_link" />
   </joint>
-  <joint
-    name="fixed_top_joint"
-    type="fixed">
+  <joint name="fixed_top_joint" type="fixed">
     <origin
       xyz="0 0 0.114485752303901"
@@ -209,7 +202,5 @@
     <child link="top_link" />
   </joint>
-  <joint
-    name="fixed_battery_joint"
-    type="fixed">
+  <joint name="fixed_battery_joint" type="fixed">
     <origin
       xyz="-0.0930197544779129 -0.00012769656788774 0"
@@ -218,7 +209,5 @@
     <child link="battery_link" />
   </joint>
-  <joint
-    name="fixed_housing_joint"
-    type="fixed">
+  <joint name="fixed_housing_joint" type="fixed">
     <origin
       xyz="0.03472949777154 0 0"
@@ -235,3 +224,58 @@
 	<xacro:wheel prefix="lb" />
 	<xacro:wheel prefix="rb" />
+<!-- Sensor -->
+  <joint name="scan_joint" type="fixed">
+    <parent link="housing_link"/>
+    <child link="scan_link"/>
+    <origin xyz="0 0 0.032" rpy="0 0 0"/>
+  </joint>
+  <link name="scan_link">
+    <visual>
+      <origin xyz="0 0 0.0" rpy="0 0 0"/>
+      <geometry>
+        <mesh filename="package://roverjw_description/meshes/sensors/lds.stl" scale="0.001 0.001 0.001"/>
+      </geometry>
+      <material name="black"/>
+    </visual>
+    <collision>
+      <origin xyz="0.015 0 -0.0065" rpy="0 0 0"/>
+      <geometry>
+        <cylinder length="0.0315" radius="0.055"/>
+      </geometry>
+    </collision>
+    <inertial>
+      <mass value="0.114" />
+      <origin xyz="0 0 0" />
+      <inertia ixx="0.001" ixy="0.0" ixz="0.0"
+               iyy="0.001" iyz="0.0"
+               izz="0.001" />
+    </inertial>
+  </link>
+  <link name="camera">
+    <collision>
+      <origin xyz="-0.0625 0 0" rpy="0 0 0"/>
+      <geometry>
+        <box size="0.025 0.05 0.025"/>
+      </geometry>
+    </collision>
+    <visual>
+      <origin xyz="-0.0625 0 0" rpy="0 0 0"/>
+      <geometry>
+        <box size="0.025 0.05 0.025"/>
+      </geometry>
+      <material name="red"/>
+    </visual>
+    <inertial>
+      <mass value="${cameraMass}" />
+      <origin xyz="0 0 0" rpy="0 0 0"/>
+      <box_inertia m="${cameraMass}" x="0.025" y="0.05" z="0.05" />
+      <inertia ixx="1e-6" ixy="0" ixz="0" iyy="1e-6" iyz="0" izz="1e-6" />
+    </inertial>
+  </link>
+  <joint name="camera_joint" type="fixed">
+    <axis xyz="0 1 0" />
+    <origin xyz=".2 0 0" rpy="0 0 0"/>
+    <parent link="housing_link"/>
+    <child link="camera"/>
+  </joint>
 </robot>

Commit message: RoverJW_slam is added

File: roverjw_description/urdf/RoverJW.xacro (robot description, xacro)
@@ -279,3 +279,21 @@
     <child link="camera"/>
   </joint>
+    <link name='imu_link'>
+      <origin xyz="0 0 0" rpy="0 0 0"/>
+    <inertial>
+      <mass value="0.015" />
+      <origin xyz="0 0 0" rpy="0 0 0"/>
+      <inertia ixx="1e-05" ixy="0.0" ixz="0.0"
+               iyy="1e-05" iyz="0.0"
+               izz="1e-05" />
+    </inertial>
+    </link>
+    <joint name="imu_joint" type="fixed">
+      <parent link="base_link"/>
+      <child link="imu_link"/>
+        <axis xyz="1 0 0" />
+        <origin xyz="0 0 0" rpy="0 0 0"/>
+        <parent link="housing_link"/>
+        <child link="camera"/>
+    </joint>
 </robot>
